File: hw/head/sigplane-head.kicad_sch (KiCad schematic)
At the start: 63 parts, among them J1 ctrl, J201 btn, J31 USB_B_Micro, J41 AudioJack3_Ground, Q111 Q_NMOS_GSD, Q121 Q_NMOS_GSD, Q131 Q_NMOS_GSD, Q3 c1815, Q31 UMH3N, Q41 ML5203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

Commit message: hw head -  элементы размещены на плате, но не соединены
Parts:
- J1: footprint Connector_JST:JST_XH_S5B-XH-A-1_1x05_P2.50mm_Horizontal -> Connector_JST:JST_XH_S5B-XH-A_1x05_P2.50mm_Horizontal
- J201: footprint Connector_JST:JST_XH_S5B-XH-A-1_1x08_P2.50mm_Horizontal -> Connector_Molex:Molex_PicoBlade_53398-0871_1x08-1MP_P1.25mm_Vertical; symbol Connector_Generic:Conn_01x08 -> Connector_Generic_MountingPin:Conn_01x08_MountingPin
- J41: value AudioJack3_Ground -> Audio out; symbol Connector_Audio:AudioJack3_Ground -> Connector_Audio:AudioJack3_SwitchT
- Q111, Q121, Q131: value Q_NMOS_GSD -> ML2502
Connections:
- net +3.3V: now also C12.1, D31.1 (K), Q41.2 (S), R41.2, U11.5 (OUT); no longer C22.2, Q31.6 (C1), R23.2, U21.3 (EN)
- net +5V: now also R44.2; no longer R44.1
- net GND: now also C22.2, C31.2, C32.1, J201.MP (MountPin), J41.TN; no longer C22.1, C31.1, C32.2, J41.G
- net VSDCARD: now also C42.1, Q41.3 (D), U41.3 (VDDIO)
- net led-b: now also R132.2; no longer R132.1
- net led-g: now also R122.2; no longer R122.1
- net led-r: now also R112.2; no longer R112.1
- net at Q3.3 (C), Q41.1 (G): now also R41.1; no longer R41.2
- net at Q121.1 (G), R123.1: now also R122.1; no longer R122.2
- net at Q131.1 (G), R133.1: now also R132.1; no longer R132.2
- net at D32.2 (A), J31.1 (VBUS), U31.7 (VREGIN)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: now also C32.2, R31.2; no longer C32.1, R31.1
- net at D31.2 (A), U31.6 (VDD): now also C31.1; no longer C31.2
- net at Q111.1 (G), R113.1: now also R112.1; no longer R112.2
- net at R32.1: now also U31.25 (RXD); no longer U31.26 (TXD)
- net at R33.1: now also U31.26 (TXD); no longer U31.25 (RXD)
- net at U31.9 (~{RST}): now also R31.1; no longer R31.2
- net at Q3.3 (C), Q43.1 (G): now also R44.1; no longer R44.2
- removed net +3V3: C12.1, D31.1 (K), Q41.2 (S), R41.1, U11.5 (OUT)
- new net s-en: C22.1, Q31.6 (C1), R23.2, U21.3 (EN)
Other:
- moved on the sheet: C22, C31, C32, R112, R122, R132, R31, R32, R33, R41, R44

Commit message: hw head -  плата разведена
Connections:
- net btn-b: now also U21.7 (IO35); no longer U21.6 (IO34)
- net btn-g: now also U21.9 (IO33); no longer U21.8 (IO32)
- net btn-r: now also U21.6 (IO34); no longer U21.7 (IO35)
- net btn-y: now also U21.8 (IO32); no longer U21.9 (IO33)
- net s-boot: now also Q31.1 (E1); no longer Q31.3 (C2)
- net s-en: now also Q31.4 (E2); no longer Q31.6 (C1)
- new net: Q31.2 (B1), Q31.3 (C2), U31.24 (~{RTS})
- new net: Q31.5 (B2), Q31.6 (C1), U31.28 (~{DTR})
Other:
- moved on the sheet: Q31A, Q31B
Changed lines of the file:
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@@
   (junction (at 43.18 160.02) (diameter 0) (color 0 0 0 0)
   )
+  (junction (at 260.35 46.99) (diameter 0) (color 0 0 0 0)
+  )
   (junction (at 101.6 173.99) (diameter 0) (color 0 0 0 0)
   )
@@
   (junction (at 182.88 86.36) (diameter 0) (color 0 0 0 0)
   )
-  (junction (at 260.35 46.99) (diameter 0) (color 0 0 0 0)
-  )
   (junction (at 120.65 181.61) (diameter 0) (color 0 0 0 0)
   )
@@
     (stroke (width 0) (type default))
   )
+  (wire (pts (xy 260.35 46.99) (xy 260.35 55.88))
+    (stroke (width 0) (type default))
+  )
   (wire (pts (xy 104.14 186.69) (xy 111.76 186.69))
     (stroke (width 0) (type default))
@@
     (stroke (width 0) (type default))
   )
-  (wire (pts (xy 260.35 46.99) (xy 260.35 40.64))
-    (stroke (width 0) (type default))
-  )
   (wire (pts (xy 142.24 133.35) (xy 153.67 133.35))
     (stroke (width 0) (type default))
@@
     (stroke (width 0) (type default))
   )
-  (wire (pts (xy 260.35 46.99) (xy 260.35 55.88))
+  (wire (pts (xy 260.35 40.64) (xy 260.35 46.99))
     (stroke (width 0) (type default))
   )
@@
     (effects (font (size 1.27 1.27)) (justify left bottom))
   )
-  (label "btn-y" (at 62.23 110.49 0) (fields_autoplaced)
+  (label "btn-y" (at 62.23 107.95 0) (fields_autoplaced)
     (effects (font (size 1.27 1.27)) (justify left bottom))
   )
@@
     (effects (font (size 1.27 1.27)) (justify left bottom))
   )
-  (label "btn-g" (at 62.23 107.95 0) (fields_autoplaced)
+  (label "btn-g" (at 62.23 110.49 0) (fields_autoplaced)
     (effects (font (size 1.27 1.27)) (justify left bottom))
   )
@@
     (effects (font (size 1.27 1.27)) (justify left bottom))
   )
-  (label "btn-r" (at 62.23 115.57 0) (fields_autoplaced)
+  (label "btn-r" (at 62.23 113.03 0) (fields_autoplaced)
     (effects (font (size 1.27 1.27)) (justify left bottom))
   )
@@
     (effects (font (size 1.27 1.27)) (justify left bottom))
   )
-  (label "btn-b" (at 62.23 113.03 0) (fields_autoplaced)
+  (label "btn-b" (at 62.23 115.57 0) (fields_autoplaced)
     (effects (font (size 1.27 1.27)) (justify left bottom))
   )
@@
     )
   )
-  (symbol (lib_id "Transistor_BJT:UMH3N") (at 265.43 62.23 0) (mirror x) (unit 1)
+  (symbol (lib_id "Transistor_BJT:UMH3N") (at 265.43 46.99 0) (mirror x) (unit 1)
     (in_bom yes) (on_board yes) (dnp no)
-    (property "Reference" "Q31" (at 273.05 60.96 0)
+    (property "Reference" "Q31" (at 273.05 45.72 0)
       (effects (font (size 1.27 1.27)) (justify left))
     )
-    (property "Value" "UMH3N" (at 273.05 63.5 0)
+    (property "Value" "UMH3N" (at 273.05 48.26 0)
       (effects (font (size 1.27 1.27)) (justify left))
     )
-    (property "Footprint" "Package_TO_SOT_SMD:SOT-363_SC-70-6" (at 265.557 51.054 0)
+    (property "Footprint" "Package_TO_SOT_SMD:SOT-363_SC-70-6" (at 265.557 35.814 0)
       (effects (font (size 1.27 1.27)) hide)
     )
-    (property "Datasheet" "http://rohmfs.rohm.com/en/products/databook/datasheet/discrete/transistor/digital/emh3t2r-e.pdf" (at 269.24 62.23 0)
+    (property "Datasheet" "http://rohmfs.rohm.com/en/products/databook/datasheet/discrete/transistor/digital/emh3t2r-e.pdf" (at 269.24 46.99 0)
       (effects (font (size 1.27 1.27)) hide)
     )
@@
     )
   )
-  (symbol (lib_id "Transistor_BJT:UMH3N") (at 265.43 46.99 0) (unit 2)
+  (symbol (lib_id "Transistor_BJT:UMH3N") (at 265.43 62.23 0) (unit 2)
     (in_bom yes) (on_board yes) (dnp no)
-    (property "Reference" "Q31" (at 273.05 45.72 0)
+    (property "Reference" "Q31" (at 273.05 60.96 0)
       (effects (font (size 1.27 1.27)) (justify left))
     )
-    (property "Value" "UMH3N" (at 273.05 48.26 0)
+    (property "Value" "UMH3N" (at 273.05 63.5 0)
       (effects (font (size 1.27 1.27)) (justify left))
     )
-    (property "Footprint" "Package_TO_SOT_SMD:SOT-363_SC-70-6" (at 265.557 58.166 0)
+    (property "Footprint" "Package_TO_SOT_SMD:SOT-363_SC-70-6" (at 265.557 73.406 0)
       (effects (font (size 1.27 1.27)) hide)
     )
-    (property "Datasheet" "http://rohmfs.rohm.com/en/products/databook/datasheet/discrete/transistor/digital/emh3t2r-e.pdf" (at 269.24 46.99 0)
+    (property "Datasheet" "http://rohmfs.rohm.com/en/products/databook/datasheet/discrete/transistor/digital/emh3t2r-e.pdf" (at 269.24 62.23 0)
       (effects (font (size 1.27 1.27)) hide)
     )
