File: hw/head/sigplane-head.kicad_pcb (KiCad board)
At the start: 2 copper layers, 95.2 x 45.1 mm, 63 parts, among them J1 ctrl, J201 btn, J31 USB_B_Micro, J41 Audio out, Q111 ML2502, Q121 ML2502, Q131 ML2502, Q31 UMH3N, Q41 ML5203, Q42 c1815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

Commit message: hw head -  плата разведена
Parts:
- moved U11 2.93 mm to (32.3, 41.0), turned to -90 degrees
- moved R21 1.02 mm to (47.5, 53.7)
- moved Q31 1.00 mm to (52.3, 54.4)
- moved C42 0.74 mm to (96.5, 31.6)
- moved C43 0.74 mm to (96.5, 37.7)
- moved Q42 0.74 mm to (86.8, 31.5)
- moved Q44 0.74 mm to (86.8, 37.7)
- moved R41 0.74 mm to (90.1, 31.5)
- moved R42 0.74 mm to (83.0, 30.7)
- moved R43 0.74 mm to (83.0, 32.9)
- moved R44 0.74 mm to (90.0, 37.7)
- moved R46 0.74 mm to (82.9, 36.9)
- moved Q41 0.74 mm to (93.3, 31.6)
- moved Q43 0.74 mm to (93.3, 37.7)
- moved U31 0.25 mm to (59.5, 56.8)
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Connections:
- Q31 pad 1: Net-(Q31A-E1) -> /s-boot
- Q31 pad 3: /s-boot -> Net-(Q31A-B1)
- Q31 pad 4: Net-(Q31A-B1) -> /s-en
- Q31 pad 5: Net-(Q31A-E1) -> Net-(Q31A-C1)
- Q31 pad 6: /s-en -> Net-(Q31A-C1)
- U21 pad 6: /btn-b -> /btn-r
- U21 pad 7: /btn-r -> /btn-b
- U21 pad 8: /btn-g -> /btn-y
- U21 pad 9: /btn-y -> /btn-g
- U31 pad 24: Net-(Q31A-E1) -> Net-(Q31A-B1)
- U31 pad 28: Net-(Q31A-B1) -> Net-(Q31A-C1)
Routing:
- net +5V: track 0.00 -> 153.4 mm, vias 0 -> 5
- net +3.3V: track 0.00 -> 119.1 mm, vias 0 -> 5
- net /led-r: track 0.00 -> 67.1 mm, vias 0 -> 3
- net /led-g: track 0.00 -> 66.8 mm, vias 0 -> 1
- net VSDCARD: track 0.00 -> 49.3 mm
- net auden: track 0.00 -> 43.4 mm, vias 0 -> 2
- net /led-b: track 0.00 -> 35.3 mm, vias 0 -> 1
- net /btn-r: track 0.00 -> 35.1 mm
- net /s-en: track 0.00 -> 32.2 mm, vias 0 -> 2
- net /btn-b: track 0.00 -> 32.2 mm
- net /btn-y: track 0.00 -> 29.1 mm
- net /aud-tx: track 0.00 -> 27.5 mm
- net /btn-g: track 0.00 -> 26.2 mm
- net Net-(U41-DACR): track 0.00 -> 25.5 mm, vias 0 -> 2
- net /s-tx: track 0.00 -> 24.7 mm, vias 0 -> 2
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- added copper zone on B.Cu, net GND
- added copper zone on F.Cu, net GND

Commit message: hw - гербер
Routing:
- net GND: vias 151 -> 165
Other:
- board text added: "sigplane-head-v0.1"
