File: hw/power/sigplane-power.kicad_pcb (KiCad board)
At the start: 2 copper layers, 47.2 x 57.4 mm, 18 parts, among them J1 ctrl, J2 led-out, J3 led-out, J4 dc-dc, J5 v-in, Q11 Q_NMOS_GSD, Q12 Q_NMOS_GSD, Q13 Q_NMOS_GSD

Commit message: hw power - изменён корпус транзистора
Parts:
- Q11, Q12, Q13: footprint Package_TO_SOT_THT:TO-220-3_Horizontal_TabDown -> Package_TO_SOT_SMD:TO-263-2
- moved Q13 26.9 mm to (69.6, 85.2)
- moved Q11 20.8 mm to (51.1, 91.7), turned to -90 degrees
- moved Q12 13.4 mm to (69.6, 97.6)
- moved R15 8.64 mm to (69.7, 72.4)
- moved R16 8.64 mm to (69.7, 75.4)
- moved R11 8.61 mm to (61.1, 72.4)
- moved R12 8.61 mm to (61.1, 75.4)
Routing:
- net /lout-r: track 40.8 -> 60.7 mm, vias 0 -> 6
- net Net-(Q13-G): track 32.2 -> 16.2 mm
- net Net-(Q11-G): track 33.2 -> 17.4 mm
- net /lout-b: track 59.0 -> 74.2 mm, vias 0 -> 5
- net /led-g: track 22.1 -> 9.34 mm
- net /led-r: track 21.9 -> 11.1 mm
- net /led-b: track 16.5 -> 8.70 mm
- net /lout-g: track 51.8 -> 48.6 mm, vias 0 -> 3
- net Net-(Q12-G): track 34.6 -> 31.9 mm
- net GND: vias 33 -> 49

Commit message: hw - гербер
Other:
- board text added: "sigplane-power-v0.1"
