File: hw/power/sigplane-power.kicad_sch (KiCad schematic)
At the start: 18 parts, among them J1 ctrl, J2 led-out, J3 led-out, J4 dc-dc, J5 v-in, Q11 Q_NMOS_GSD, Q12 Q_NMOS_GSD, Q13 Q_NMOS_GSD

Commit message: hw power - изменён корпус транзистора
Parts:
- Q11, Q12, Q13: footprint Package_TO_SOT_THT:TO-220-3_Horizontal_TabDown -> Package_TO_SOT_SMD:TO-263-2
Changed lines of the file:
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@@
       (effects (font (size 1.27 1.27)) (justify left))
     )
-    (property "Footprint" "Package_TO_SOT_THT:TO-220-3_Horizontal_TabDown" (at 66.04 58.42 0)
+    (property "Footprint" "Package_TO_SOT_SMD:TO-263-2" (at 66.04 58.42 0)
       (effects (font (size 1.27 1.27)) hide)
     )
@@
       (effects (font (size 1.27 1.27)) (justify left))
     )
-    (property "Footprint" "Package_TO_SOT_THT:TO-220-3_Horizontal_TabDown" (at 66.04 77.47 0)
+    (property "Footprint" "Package_TO_SOT_SMD:TO-263-2" (at 66.04 77.47 0)
       (effects (font (size 1.27 1.27)) hide)
     )
@@
       (effects (font (size 1.27 1.27)) (justify left))
     )
-    (property "Footprint" "Package_TO_SOT_THT:TO-220-3_Horizontal_TabDown" (at 66.04 96.52 0)
-      (effects (font (size 1.27 1.27)) hide)
-    )
+    (property "Footprint" "Package_TO_SOT_SMD:TO-263-2" (at 66.04 96.52 0)
+      (effects (font (size 1.27 1.27)) hide)
+    )

Commit message: hw - гербер
Parts:
- Q11, Q12, Q13: value Q_NMOS_GSD -> IRL3705NS
Changed lines of the file:
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@@
       (effects (font (size 1.27 1.27)) (justify left))
     )
-    (property "Value" "Q_NMOS_GSD" (at 67.31 62.23 0)
+    (property "Value" "IRL3705NS" (at 67.31 62.23 0)
       (effects (font (size 1.27 1.27)) (justify left))
     )
@@
       (effects (font (size 1.27 1.27)) (justify left))
     )
-    (property "Value" "Q_NMOS_GSD" (at 67.31 81.28 0)
+    (property "Value" "IRL3705NS" (at 67.31 81.28 0)
       (effects (font (size 1.27 1.27)) (justify left))
     )
@@
       (effects (font (size 1.27 1.27)) (justify left))
     )
-    (property "Value" "Q_NMOS_GSD" (at 67.31 100.33 0)
-      (effects (font (size 1.27 1.27)) (justify left))
-    )
+    (property "Value" "IRL3705NS" (at 67.31 100.33 0)
+      (effects (font (size 1.27 1.27)) (justify left))
+    )
